Commit message: part3

File: barista_robot_description/xacro/barista_robot_model.urdf.xacro (robot description, xacro)
@@ -54,57 +54,2 @@
 <xacro:top_joint origin_xyz="0.0 0.0 0.3425" origin_rpy="0 0 1.57" />
 </robot>
-<?xml version="1.0" ?>
-<robot name="barista" xmlns:xacro="http://www.ros.org/wiki/xacro">
-  <!-- Include external files -->
-  <xacro:include filename="$(find barista_robot_description)/xacro/wheel.xacro"/>
-  <xacro:include filename="$(find barista_robot_description)/xacro/standoff.xacro"/>
-  <xacro:include filename="$(find barista_robot_description)/xacro/laser_scanner.xacro"/>
-  <xacro:include filename="$(find barista_robot_description)/xacro/cup_holder_tray.xacro"/>
-  <!-- Define the base link of the robot -->
-  <link name="base_link">
-    <!-- Visual representation of the base link -->
-    <visual>
-      <geometry>
-        <cylinder length="0.155" radius="0.178"/>
-      </geometry>
-    </visual>
-    <!-- Inertial properties of the base link -->
-    <inertial>
-      <mass value="10.0"/>
-      <inertia ixx="1.0" ixy="0.0" ixz="0.0" iyy="1.0" iyz="0.0" izz="1.0"/>
-    </inertial>
-    <!-- Collision representation of the base link -->
-    <collision>
-      <geometry>
-        <cylinder length="0.155" radius="0.178"/>
-      </geometry>
-    </collision>
-  </link>
-  <!-- Gazebo-specific configuration for the base link -->
-  <gazebo reference="base_link">
-    <material>Gazebo/Green</material>
-  </gazebo>
-  <!-- Include and instantiate the wheel.xacro macro for the left wheel -->
-  <xacro:wheel prefix="left" />
-<xacro:wheel_color prefix="left" />
-  <!-- Include and instantiate the joint_wheel.xacro macro for the left wheel joint -->
-  <xacro:joint_wheel prefix="left" x="0.1" />
-  <!-- Include and instantiate the wheel.xacro macro for the right wheel -->
-  <xacro:wheel prefix="right" />
-<xacro:wheel_color prefix="right" />
-  <!-- Include and instantiate the joint_wheel.xacro macro for the right wheel joint -->
-  <xacro:joint_wheel prefix="right" x="-0.1" />
-  <xacro:standoff_link prefix="stand1" />
-  <xacro:standoff_joint prefix="stand1" x="0.1" y="0.1" z="0.185" />
-<xacro:standoff_link prefix="stand2" />
-<xacro:standoff_joint prefix="stand2" x="0.1" y="-0.1" z="0.185" />
-<xacro:standoff_link prefix="stand3" />
-<xacro:standoff_joint prefix="stand3" x="-0.1" y="0.1" z="0.185" />
-<xacro:standoff_link prefix="stand4" />
-<xacro:standoff_joint prefix="stand4" x="-0.1" y="-0.1" z="0.185" />
-<xacro:laser_scanner />
-<xacro:laser_scan_joint />
-<xacro:laser_plugin />
-<xacro:top />
-<xacro:top_joint origin_xyz="0.0 0.0 0.3425" origin_rpy="0 0 1.57" />
-</robot>
