Commit message: part3 done and improved

File: barista_robot_description/urdf/barista_robot_model.urdf (robot description, URDF)
Before this commit: robot baristabot, 9 links, 8 joints
Links:
- added link c1, mass 0.05; collision sphere radius=0.0352; visual sphere radius=0.0352
- added link c2, mass 0.05; collision sphere radius=0.0352; visual sphere radius=0.0352
Joints:
- added joint c1_joint: type fixed, parent base_link, child c1, origin xyz=0.0 -0.1  -0.09 rpy=0 1.57 0
- added joint c2_joint: type fixed, parent base_link, child c2, origin xyz=0.0 0.1  -0.09 rpy=0 1.57 0

File: barista_robot_description/xacro/barista.urdf.xacro (robot description, xacro)
@@ -38,4 +38,48 @@
 <xacro:wheel_color prefix="right" />
   <xacro:joint_wheel prefix="right" x="-0.1" />
+<link name="c1">
+    <visual>
+      <geometry>
+        <sphere radius="0.0352"/>
+      </geometry>
+      <material name="castor_color"/>
+    </visual>
+        <inertial>
+      <mass value="0.05"/>
+      <inertia ixx="1.0" ixy="0.0" ixz="0.0" iyy="1.0" iyz="0.0" izz="1.0"/>
+    </inertial>
+         <collision>
+      <geometry>
+       <sphere radius="0.0352"/>
+      </geometry>
+      </collision>
+</link>
+  <joint name="c1_joint" type="fixed">
+    <parent link="base_link"/>
+    <child link="c1"/>
+    <origin xyz="0.0 -0.1  -0.09" rpy="0 1.57 0" />
+  </joint>
+<link name="c2">
+    <visual>
+      <geometry>
+        <sphere radius="0.0352"/>
+      </geometry>
+      <material name="castor_color"/>
+    </visual>
+        <inertial>
+      <mass value="0.05"/>
+      <inertia ixx="1.0" ixy="0.0" ixz="0.0" iyy="1.0" iyz="0.0" izz="1.0"/>
+    </inertial>
+         <collision>
+      <geometry>
+       <sphere radius="0.0352"/>
+      </geometry>
+      </collision>
+</link>
+  <joint name="c2_joint" type="fixed">
+    <parent link="base_link"/>
+    <child link="c2"/>
+    <origin xyz="0.0 0.1  -0.09" rpy="0 1.57 0" />
+  </joint>
   <gazebo>
     <plugin name="diff_drive" filename="libgazebo_ros_diff_drive.so">

File: barista_robot_description/xacro/barista_2.urdf.xacro (robot description, xacro)
@@ -32,4 +32,48 @@
     <material>Gazebo/Green</material>
   </gazebo>
+<link name="c1">
+    <visual>
+      <geometry>
+        <sphere radius="0.0352"/>
+      </geometry>
+      <material name="castor_color"/>
+    </visual>
+        <inertial>
+      <mass value="0.05"/>
+      <inertia ixx="1.0" ixy="0.0" ixz="0.0" iyy="1.0" iyz="0.0" izz="1.0"/>
+    </inertial>
+         <collision>
+      <geometry>
+       <sphere radius="0.0352"/>
+      </geometry>
+      </collision>
+</link>
+  <joint name="c1_joint" type="fixed">
+    <parent link="base_link"/>
+    <child link="c1"/>
+    <origin xyz="0.0 -0.1  -0.09" rpy="0 1.57 0" />
+  </joint>
+<link name="c2">
+    <visual>
+      <geometry>
+        <sphere radius="0.0352"/>
+      </geometry>
+      <material name="castor_color"/>
+    </visual>
+        <inertial>
+      <mass value="0.05"/>
+      <inertia ixx="1.0" ixy="0.0" ixz="0.0" iyy="1.0" iyz="0.0" izz="1.0"/>
+    </inertial>
+         <collision>
+      <geometry>
+       <sphere radius="0.0352"/>
+      </geometry>
+      </collision>
+</link>
+  <joint name="c2_joint" type="fixed">
+    <parent link="base_link"/>
+    <child link="c2"/>
+    <origin xyz="0.0 0.1  -0.09" rpy="0 1.57 0" />
+  </joint>
   <!-- Include and instantiate the wheel.xacro macro for the left wheel -->
   <xacro:wheel prefix="left" />
